File: Fuji-Handheld/Fuji-Handheld.kicad_sch (KiCad schematic)
At the start: 0 parts

Commit message: schematic v1.0
Parts:
- added C1, C2: 4.7uF, symbol Device:C
- added C3, C4, C6: 10uF, symbol Device:C
- added C5: 1uF, symbol Device:C
- added C7, C8: 100nF, symbol Device:C
- added D1: LED, symbol Device:LED
- added J1: USB_C_Receptacle_USB2.0_16P, symbol Connector:USB_C_Receptacle_USB2.0_16P
- added J2: Conn_01x02_Pin, symbol Connector:Conn_01x02_Pin
- added J3: Conn_01x08_Pin, symbol Connector:Conn_01x08_Pin
- added JP1: SolderJumper_2_Bridged, symbol Jumper:SolderJumper_2_Bridged
- added R1, R2: 5.1k, symbol Device:R
- added R3: 4k, symbol Device:R
- added R4: 1k, symbol Device:R
- added R5, R6: 10k, symbol Device:R
- added R7, R8: 100k, symbol Device:R
- added SW1: SW_SPDT, symbol Switch:SW_SPDT
- added SW2, SW3, SW4, SW5, SW6, SW7, SW8, SW9: SW_Push, symbol Switch:SW_Push
- added U1: MCP73831-2-OT, Package_TO_SOT_SMD:SOT-23-5, symbol Battery_Management:MCP73831-2-OT
- added U2: AP2112K-3.3, Package_TO_SOT_SMD:SOT-23-5, symbol Regulator_Linear:AP2112K-3.3
- added U3: ESP32-S3-MINI-1, RF_Module:ESP32-S2-MINI-1, symbol RF_Module:ESP32-S3-MINI-1
Connections:
- new net: D1.1 (K), U1.1 (STAT)
- new net: R3.2, U1.5 (PROG)
- new net: R6.1, SW3.2, U3.4 (IO0)
- new net: J3.8 (Pin_8), JP1.1 (A)
- new net: J1.A5 (CC1), R1.1
- new net: J1.B5 (CC2), R2.2
- new net: D1.2 (A), R4.1
- new net: C5.2, R5.1, SW2.2, U3.45 (EN)
- new net +3V3: C4.2, C6.2, C8.2, J3.2 (Pin_2), JP1.2 (B), R5.2, R6.2, U2.5 (VOUT), U3.3 (3V3)
- new net +BAT: C1.2, J2.1 (Pin_1), SW1.2 (B), U1.3 (V_{BAT})
- new net BTN_A: SW8.1, U3.10 (IO6)
- new net BTN_B: SW9.1, U3.19 (IO15)
- new net BTN_DOWN: SW5.1, U3.6 (IO2)
- new net BTN_LEFT: SW6.1, U3.8 (IO4)
- new net BTN_RIGHT: SW7.1, U3.9 (IO5)
- new net BTN_UP: SW4.1, U3.5 (IO1)
- new net GND: C1.1, C2.1, C3.1, C4.1, C5.1, C6.1, C7.1, C8.1, J1.A1 (GND), J1.A12 (GND), J1.B1 (GND), J1.B12 (GND), J1.SH (SHIELD), J2.2 (Pin_2), J3.1 (Pin_1), R1.2, R2.1, R3.1, R8.2, SW2.1, SW3.1, SW4.2, SW5.2, SW6.2, SW7.2, SW8.2, SW9.2, U1.2 (V_{SS}), U2.2 (GND), U3.1 (GND), U3.2 (GND), U3.42 (GND), U3.43 (GND), U3.46 (GND), U3.47 (GND), U3.48 (GND), U3.49 (GND), U3.50 (GND), U3.51 (GND), U3.52 (GND), U3.53 (GND), U3.54 (GND), U3.55 (GND), U3.56 (GND), U3.57 (GND), U3.58 (GND), U3.59 (GND), U3.60 (GND), U3.61 (GND), U3.62 (GND), U3.63 (GND), U3.64 (GND), U3.65 (GND)
- new net TFT_CS: J3.7 (Pin_7), U3.14 (IO10)
- new net TFT_DC: J3.6 (Pin_6), U3.13 (IO9)
- new net TFT_MOSI: J3.4 (Pin_4), U3.15 (IO11)
- new net TFT_RST: J3.5 (Pin_5), U3.12 (IO8)
- new net TFT_SCLK: J3.3 (Pin_3), U3.16 (IO12)
- new net USB_DN: J1.A7 (D-), J1.B7 (D-), U3.23 (USB_D-)
- new net USB_DP: J1.A6 (D+), J1.B6 (D+), U3.24 (USB_D+)
- new net VBAT_SENSE: C7.2, R7.2, R8.1, U3.18 (IO14)
- new net VBUS: C2.2, J1.A4 (VBUS), J1.A9 (VBUS), J1.B4 (VBUS), J1.B9 (VBUS), R4.2, U1.4 (V_{DD})
- new net VSYS: C3.2, R7.1, SW1.1 (A), U2.1 (VIN), U2.3 (EN)
- no-connect marks 0 -> 27
Other:
- note added: "3.3V regulator (SW1 + U2)"
- note added: "Battery Managment (R7-8, C7)"
- note added: "Buttons (SW4-9)"
- note added: "Charger (U1 + J2)"
- note added: "Display (J3)"
- note added: "ESP32 (U3)"
- note added: "USB (J1)"

Commit message: PCB routing pt 2
Parts:
- C1, C2, C3, C4, C5, C6, C7, C8: footprint (none) -> Capacitor_SMD:C_0805_2012Metric_Pad1.18x1.45mm_HandSolder
- D1: footprint (none) -> LED_THT:LED_D3.0mm
- J1: footprint (none) -> Connector_USB:USB_C_Receptacle_HRO_TYPE-C-31-M-12
- J2: footprint (none) -> Connector_JST:JST_PH_B2B-PH-K_1x02_P2.00mm_Vertical
- J3: footprint (none) -> Connector_PinHeader_2.54mm:PinHeader_1x08_P2.54mm_Vertical
- JP1: footprint (none) -> Jumper:SolderJumper-2_P1.3mm_Bridged_RoundedPad1.0x1.5mm
- R1, R2, R3, R4, R5, R6, R7, R8: footprint (none) -> Resistor_SMD:R_0805_2012Metric_Pad1.20x1.40mm_HandSolder
- SW1: footprint (none) -> Button_Switch_SMD:SW_SPDT_PCM12
- SW2, SW3, SW4, SW5, SW6, SW7, SW8, SW9: footprint (none) -> Button_Switch_THT:SW_PUSH_6mm_H4.3mm
Changed lines of the file:
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@@
 			)
 		)
-		(property "Footprint" ""
+		(property "Footprint" "Button_Switch_THT:SW_PUSH_6mm_H4.3mm"
 			(at 200.66 110.49 0)
 			(hide yes)
@@
 			)
 		)
-		(property "Footprint" ""
+		(property "Footprint" "Resistor_SMD:R_0805_2012Metric_Pad1.20x1.40mm_HandSolder"
 			(at 88.9 106.172 90)
 			(hide yes)
@@
 			)
 		)
-		(property "Footprint" ""
+		(property "Footprint" "Capacitor_SMD:C_0805_2012Metric_Pad1.18x1.45mm_HandSolder"
 			(at 204.47 25.7048 0)
 			(hide yes)
@@
 			)
 		)
-		(property "Footprint" ""
+		(property "Footprint" "Capacitor_SMD:C_0805_2012Metric_Pad1.18x1.45mm_HandSolder"
 			(at 115.2652 78.74 0)
 			(hide yes)
@@
 			)
 		)
-		(property "Footprint" ""
+		(property "Footprint" "Button_Switch_THT:SW_PUSH_6mm_H4.3mm"
 			(at 170.18 45.72 0)
 			(hide yes)
@@
 			)
 		)
-		(property "Footprint" ""
+		(property "Footprint" "Button_Switch_THT:SW_PUSH_6mm_H4.3mm"
 			(at 168.91 105.41 0)
 			(hide yes)
@@
 			)
 		)
-		(property "Footprint" ""
+		(property "Footprint" "Jumper:SolderJumper-2_P1.3mm_Bridged_RoundedPad1.0x1.5mm"
 			(at 128.27 118.11 0)
 			(hide yes)
@@
 			)
 		)
-		(property "Footprint" ""
+		(property "Footprint" "Connector_USB:USB_C_Receptacle_HRO_TYPE-C-31-M-12"
 			(at 38.1 41.91 0)
 			(hide yes)
@@
 			)
 		)
-		(property "Footprint" ""
+		(property "Footprint" "LED_THT:LED_D3.0mm"
 			(at 121.92 40.64 0)
 			(hide yes)
@@
 			)
 		)
-		(property "Footprint" ""
+		(property "Footprint" "Button_Switch_SMD:SW_SPDT_PCM12"
 			(at 88.9 77.47 0)
 			(hide yes)
@@
 			)
 		)
-		(property "Footprint" ""
+		(property "Footprint" "Capacitor_SMD:C_0805_2012Metric_Pad1.18x1.45mm_HandSolder"
 			(at 209.55 27.6352 0)
 			(hide yes)
@@
 			)
 		)
-		(property "Footprint" ""
+		(property "Footprint" "Button_Switch_THT:SW_PUSH_6mm_H4.3mm"
 			(at 182.88 30.48 0)
 			(hide yes)
@@
 			)
 		)
-		(property "Footprint" ""
+		(property "Footprint" "Resistor_SMD:R_0805_2012Metric_Pad1.20x1.40mm_HandSolder"
 			(at 171.45 38.862 90)
 			(hide yes)
@@
 			)
 		)
-		(property "Footprint" ""
+		(property "Footprint" "Button_Switch_THT:SW_PUSH_6mm_H4.3mm"
 			(at 229.87 105.41 0)
 			(hide yes)
@@
 			)
 		)
-		(property "Footprint" ""
+		(property "Footprint" "Resistor_SMD:R_0805_2012Metric_Pad1.20x1.40mm_HandSolder"
 			(at 90.17 42.418 90)
 			(hide yes)
@@
 			)
 		)
-		(property "Footprint" ""
+		(property "Footprint" "Resistor_SMD:R_0805_2012Metric_Pad1.20x1.40mm_HandSolder"
 			(at 88.9 102.108 90)
 			(hide yes)
@@
 			)
 		)
-		(property "Footprint" ""
+		(property "Footprint" "Button_Switch_THT:SW_PUSH_6mm_H4.3mm"
 			(at 168.91 110.49 0)
 			(hide yes)
@@
 			)
 		)
-		(property "Footprint" ""
+		(property "Footprint" "Resistor_SMD:R_0805_2012Metric_Pad1.20x1.40mm_HandSolder"
 			(at 53.34 32.512 90)
 			(hide yes)
@@
 			)
 		)
-		(property "Footprint" ""
+		(property "Footprint" "Resistor_SMD:R_0805_2012Metric_Pad1.20x1.40mm_HandSolder"
 			(at 161.29 33.782 90)
 			(hide yes)
@@
 			)
 		)
-		(property "Footprint" ""
+		(property "Footprint" "Connector_PinHeader_2.54mm:PinHeader_1x08_P2.54mm_Vertical"
 			(at 118.11 107.95 0)
 			(hide yes)
@@
 			)
 		)
-		(property "Footprint" ""
+		(property "Footprint" "Button_Switch_THT:SW_PUSH_6mm_H4.3mm"
 			(at 200.66 105.41 0)
 			(hide yes)
@@
 			)
 		)
-		(property "Footprint" ""
+		(property "Footprint" "Button_Switch_THT:SW_PUSH_6mm_H4.3mm"
 			(at 229.87 110.49 0)
 			(hide yes)
@@
 			)
 		)
-		(property "Footprint" ""
+		(property "Footprint" "Capacitor_SMD:C_0805_2012Metric_Pad1.18x1.45mm_HandSolder"
 			(at 104.14 28.9052 0)
 			(hide yes)
@@
 			)
 		)
-		(property "Footprint" ""
+		(property "Footprint" "Capacitor_SMD:C_0805_2012Metric_Pad1.18x1.45mm_HandSolder"
 			(at 92.71 115.8748 0)
 			(hide yes)
@@
 			)
 		)
-		(property "Footprint" ""
+		(property "Footprint" "Capacitor_SMD:C_0805_2012Metric_Pad1.18x1.45mm_HandSolder"
 			(at 135.5852 78.74 0)
 			(hide yes)
@@
 			)
 		)
-		(property "Footprint" ""
+		(property "Footprint" "Resistor_SMD:R_0805_2012Metric_Pad1.20x1.40mm_HandSolder"
 			(at 130.81 42.418 90)
 			(hide yes)
@@
 			)
 		)
-		(property "Footprint" ""
+		(property "Footprint" "Capacitor_SMD:C_0805_2012Metric_Pad1.18x1.45mm_HandSolder"
 			(at 124.1552 35.56 0)
 			(hide yes)
@@
 			)
 		)
-		(property "Footprint" ""
+		(property "Footprint" "Resistor_SMD:R_0805_2012Metric_Pad1.20x1.40mm_HandSolder"
 			(at 53.34 33.528 90)
 			(hide yes)
@@
 			)
 		)
-		(property "Footprint" ""
+		(property "Footprint" "Capacitor_SMD:C_0805_2012Metric_Pad1.18x1.45mm_HandSolder"
 			(at 169.8752 35.56 0)
 			(hide yes)
@@
 			)
 		)
-		(property "Footprint" ""
+		(property "Footprint" "Connector_JST:JST_PH_B2B-PH-K_1x02_P2.00mm_Vertical"
 			(at 116.84 54.61 0)
 			(hide yes)

Commit message: Finished with the pcb / gerber files
Parts:
- SW2, SW3: footprint Button_Switch_THT:SW_PUSH_6mm_H4.3mm -> Button_Switch_SMD:SW_SPST_PTS810
Changed lines of the file:
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@@
 			)
 		)
-		(property "Footprint" "Button_Switch_THT:SW_PUSH_6mm_H4.3mm"
+		(property "Footprint" "Button_Switch_SMD:SW_SPST_PTS810"
 			(at 170.18 45.72 0)
 			(hide yes)
@@
 			)
 		)
-		(property "Footprint" "Button_Switch_THT:SW_PUSH_6mm_H4.3mm"
+		(property "Footprint" "Button_Switch_SMD:SW_SPST_PTS810"
 			(at 182.88 30.48 0)
 			(hide yes)
